Commit message: 更改URDF命名

File: resources/robots/my_legged/urdf/urdf.urdf (robot description, URDF)
Before this commit: robot urdf, 11 links, 10 joints
Links:
- link L1: geometry collision mesh filename=../meshes/L1.STL; visual mesh filename=../meshes/L1.STL
- link L2: geometry collision mesh filename=../meshes/L2.STL; visual mesh filename=../meshes/L2.STL
- link L3: geometry collision mesh filename=../meshes/L3.STL; visual mesh filename=../meshes/L3.STL
- link L4: geometry collision mesh filename=../meshes/L4.STL; visual mesh filename=../meshes/L4.STL
- link L5: geometry collision mesh filename=../meshes/L5.STL; visual mesh filename=../meshes/L5.STL
- link R1: geometry collision mesh filename=../meshes/R1.STL; visual mesh filename=../meshes/R1.STL
- link R2: geometry collision mesh filename=../meshes/R2.STL; visual mesh filename=../meshes/R2.STL
- link R3: geometry collision mesh filename=../meshes/R3.STL; visual mesh filename=../meshes/R3.STL
- link R4: geometry collision mesh filename=../meshes/R4.STL; visual mesh filename=../meshes/R4.STL
- link R5: geometry collision mesh filename=../meshes/R5.STL; visual mesh filename=../meshes/R5.STL
- link base_link: geometry collision mesh filename=../meshes/base_link.STL; visual mesh filename=../meshes/base_link.STL
Joints:
- removed joint jl1
- removed joint jl2
- removed joint jl3
- removed joint jl4
- removed joint jl5
- removed joint jr1
- removed joint jr2
- removed joint jr3
- removed joint jr4
- removed joint jr5
- added joint left_ankle_pitch_joint: type revolute, parent L3, child L4, origin xyz=-0.311 -0.003 0 rpy=0 0 0, axis 0 1 0, limit lower=-2 upper=2 effort=100 velocity=50
- added joint left_ankle_roll_joint: type revolute, parent L4, child L5, origin xyz=0 0 0 rpy=0 0 0, axis 0 0 1, limit lower=-2 upper=2 effort=100 velocity=50
- added joint left_hip_pitch_joint: type revolute, parent L1, child L2, origin xyz=0 0 0 rpy=0 0 0, axis 0 1 0, limit lower=-2 upper=2 effort=100 velocity=50
- added joint left_hip_yaw_joint: type revolute, parent base_link, child L1, origin xyz=0 -0.0785 0 rpy=0 0 0, axis 0 0 1, limit lower=-2 upper=2 effort=100 velocity=50
- added joint left_knee_pitch_joint: type revolute, parent L2, child L3, origin xyz=-0.3 0 0 rpy=0 0 0, axis 0 1 0, limit lower=-2 upper=2 effort=100 velocity=50
- added joint right_ankle_pitch_joint: type revolute, parent R3, child R4, origin xyz=-0.311 0 0 rpy=0 0 0, axis 0 1 0, limit lower=-2 upper=2 effort=100 velocity=50
- added joint right_ankle_roll_joint: type revolute, parent R4, child R5, origin xyz=0 0 0 rpy=0 0 0, axis 0 0 1, limit lower=-2 upper=2 effort=100 velocity=50
- added joint right_hip_pitch_joint: type revolute, parent R1, child R2, origin xyz=0 0 0 rpy=0 0 0, axis 0 1 0, limit lower=-2 upper=2 effort=100 velocity=50
- added joint right_hip_yaw_joint: type revolute, parent base_link, child R1, origin xyz=0 0.0815 0 rpy=0 0 0, axis 0 0 1, limit lower=-2 upper=2 effort=100 velocity=50
- added joint right_knee_pitch_joint: type revolute, parent R2, child R3, origin xyz=-0.3 0 0 rpy=0 0 0, axis 0 1 0, limit lower=-2 upper=2 effort=100 velocity=50

Commit message: 更改一部分变换模型后的；张量维度错误

File: resources/robots/my_legged/urdf/urdf.urdf (robot description, URDF)
Before this commit: robot urdf, 11 links, 10 joints
Links:
- removed link L1
- removed link L2
- removed link L3
- removed link L4
- removed link L5
- removed link R1
- removed link R2
- removed link R3
- removed link R4
- removed link R5
- added link left_ankle_pitch, mass 0.019465; collision mesh filename=../meshes/left_ankle_pitch.STL; visual mesh filename=../meshes/left_ankle_pitch.STL
- added link left_ankle_roll, mass 0.27177; collision mesh filename=../meshes/left_ankle_roll.STL; visual mesh filename=../meshes/left_ankle_roll.STL
- added link left_hip_pitch, mass 1.6236; collision mesh filename=../meshes/left_hip_pitch.STL; visual mesh filename=../meshes/left_hip_pitch.STL
- added link left_hip_yaw, mass 0.59683; collision mesh filename=../meshes/left_hip_yaw.STL; visual mesh filename=../meshes/left_hip_yaw.STL
- added link left_knee_pitch, mass 0.24651; collision mesh filename=../meshes/left_knee_pitch.STL; visual mesh filename=../meshes/left_knee_pitch.STL
- added link right_ankle_pitch, mass 0.019465; collision mesh filename=../meshes/right_ankle_pitch.STL; visual mesh filename=../meshes/right_ankle_pitch.STL
- added link right_ankle_roll, mass 0.27177; collision mesh filename=../meshes/right_ankle_roll.STL; visual mesh filename=../meshes/right_ankle_roll.STL
- added link right_hip_pitch, mass 1.6182; collision mesh filename=../meshes/right_hip_pitch.STL; visual mesh filename=../meshes/right_hip_pitch.STL
- added link right_hip_yaw, mass 0.59683; collision mesh filename=../meshes/right_hip_yaw.STL; visual mesh filename=../meshes/right_hip_yaw.STL
- added link right_knee_pitch, mass 0.24651; collision mesh filename=../meshes/right_knee_pitch.STL; visual mesh filename=../meshes/right_knee_pitch.STL
Joints:
- joint left_ankle_pitch_joint: child L4 -> left_ankle_pitch; parent L3 -> left_knee_pitch
- joint left_ankle_roll_joint: child L5 -> left_ankle_roll; parent L4 -> left_ankle_pitch
- joint left_hip_pitch_joint: child L2 -> left_hip_pitch; parent L1 -> left_hip_yaw
- joint left_hip_yaw_joint: child L1 -> left_hip_yaw
- joint left_knee_pitch_joint: child L3 -> left_knee_pitch; parent L2 -> left_hip_pitch
- joint right_ankle_pitch_joint: child R4 -> right_ankle_pitch; parent R3 -> right_knee_pitch
- joint right_ankle_roll_joint: child R5 -> right_ankle_roll; parent R4 -> right_ankle_pitch
- joint right_hip_pitch_joint: child R2 -> right_hip_pitch; parent R1 -> right_hip_yaw
- joint right_hip_yaw_joint: child R1 -> right_hip_yaw
- joint right_knee_pitch_joint: child R3 -> right_knee_pitch; parent R2 -> right_hip_pitch

Commit message: 修改URDF文件，从卧姿改为站姿

File: resources/robots/my_legged/urdf/urdf.urdf (robot description, URDF)
Before this commit: robot urdf, 11 links, 10 joints
Joints:
- joint left_hip_pitch_joint: origin xyz=0 0 0 rpy=0 0 0 -> xyz=0 0 0 rpy=0 -1.5708 0
- joint left_hip_yaw_joint: axis 0 0 1 -> 1 0 0
- joint right_hip_yaw_joint: origin xyz=0 0.0815 0 rpy=0 0 0 -> xyz=0 0.0815 0 rpy=0 -1.57 0

Commit message: 修改错误的关节命名

File: resources/robots/my_legged/urdf/urdf.urdf (robot description, URDF)
Before this commit: robot urdf, 11 links, 10 joints
Links:
- removed link left_hip_yaw
- removed link right_hip_yaw
- added link left_hip_roll, mass 0.59683; collision mesh filename=../meshes/left_hip_roll.STL; visual mesh filename=../meshes/left_hip_roll.STL
- added link right_hip_roll, mass 0.59683; collision mesh filename=../meshes/right_hip_roll.STL; visual mesh filename=../meshes/right_hip_roll.STL
Joints:
- removed joint left_hip_yaw_joint
- removed joint right_hip_yaw_joint
- added joint left_hip_roll_joint: type revolute, parent base_link, child left_hip_roll, origin xyz=0 -0.0785 0 rpy=0 0 0, axis 1 0 0, limit lower=-2 upper=2 effort=100 velocity=50
- added joint right_hip_roll_joint: type revolute, parent base_link, child right_hip_roll, origin xyz=0 0.0815 0 rpy=0 -1.57 0, axis 0 0 1, limit lower=-2 upper=2 effort=100 velocity=50
- joint left_hip_pitch_joint: parent left_hip_yaw -> left_hip_roll
- joint right_hip_pitch_joint: parent right_hip_yaw -> right_hip_roll

Commit message: 修改URDF文件和参数等

File: resources/robots/my_legged/urdf/urdf.urdf (robot description, URDF)
Before this commit: robot urdf, 11 links, 10 joints
Joints:
- joint left_ankle_pitch_joint: limit lower=-2 upper=2 effort=100 velocity=50 -> lower=-0.5 upper=0.5 effort=100 velocity=50
- joint left_ankle_roll_joint: limit lower=-2 upper=2 effort=100 velocity=50 -> lower=-0.4 upper=0.4 effort=100 velocity=50
- joint left_hip_pitch_joint: limit lower=-2 upper=2 effort=100 velocity=50 -> lower=-0.5 upper=0.9 effort=100 velocity=50
- joint left_hip_roll_joint: limit lower=-2 upper=2 effort=100 velocity=50 -> lower=-0.8 upper=0.2 effort=100 velocity=50
- joint left_knee_pitch_joint: limit lower=-2 upper=2 effort=100 velocity=50 -> lower=-1.5 upper=0 effort=100 velocity=50
- joint right_ankle_pitch_joint: limit lower=-2 upper=2 effort=100 velocity=50 -> lower=-0.5 upper=0.5 effort=100 velocity=50
- joint right_ankle_roll_joint: limit lower=-2 upper=2 effort=100 velocity=50 -> lower=-0.4 upper=0.4 effort=100 velocity=50
- joint right_hip_pitch_joint: limit lower=-2 upper=2 effort=100 velocity=50 -> lower=-0.5 upper=0.9 effort=100 velocity=50
- joint right_hip_roll_joint: limit lower=-2 upper=2 effort=100 velocity=50 -> lower=-0.8 upper=0.2 effort=100 velocity=50
- joint right_knee_pitch_joint: limit lower=-2 upper=2 effort=100 velocity=50 -> lower=-1.5 upper=0 effort=100 velocity=50

Commit message: 修改urdf文件配置问题

File: resources/robots/my_legged/urdf/urdf.urdf (robot description, URDF)
Before this commit: robot urdf, 11 links, 10 joints
Joints:
- joint left_ankle_pitch_joint: axis 0 1 0 -> 0 -1 0
- joint left_knee_pitch_joint: axis 0 1 0 -> 0 -1 0; limit lower=-1.5 upper=0 effort=100 velocity=50 -> lower=0 upper=1.5 effort=100 velocity=50
- joint right_ankle_pitch_joint: axis 0 1 0 -> 0 -1 0
- joint right_hip_pitch_joint: axis 0 1 0 -> 0 -1 0; limit lower=-0.5 upper=0.9 effort=100 velocity=50 -> lower=-0.9 upper=0.5 effort=100 velocity=50
- joint right_knee_pitch_joint: axis 0 1 0 -> 0 -1 0; limit lower=-1.5 upper=0 effort=100 velocity=50 -> lower=0 upper=1.5 effort=100 velocity=50
